Commit message: save tmp

File: jaka_robot_v2.2/src/jaka_zu7_moveit_config/config/jaka_zu7.ros2_control.xacro (robot description, xacro)
@@ -6,7 +6,8 @@
             <hardware>
                 <!-- By default, set up controllers for simulation. This won't work on real hardware -->
-                <plugin>mock_components/GenericSystem</plugin>
+                <!-- <plugin>mock_components/GenericSystem</plugin> -->
+                <plugin>jaka_hardware/JAKAHardwareInterface</plugin>
             </hardware>
-            <joint name="joint_1">
+            <!-- <joint name="joint_1">
                 <command_interface name="position"/>
                 <state_interface name="position">
@@ -49,5 +50,5 @@
                 </state_interface>
                 <state_interface name="velocity"/>
-            </joint>
+            </joint> -->
         </ros2_control>
     </xacro:macro>

Commit message: use JAKAHardwareInterface in jaka_zu7.ros2_control.xacro

File: jaka_robot_v2.2/src/jaka_zu7_moveit_config/config/jaka_zu7.ros2_control.xacro (robot description, xacro)
@@ -9,5 +9,5 @@
                 <plugin>jaka_hardware/JAKAHardwareInterface</plugin>
             </hardware>
-            <!-- <joint name="joint_1">
+            <joint name="joint_1">
                 <command_interface name="position"/>
                 <state_interface name="position">
@@ -50,5 +50,5 @@
                 </state_interface>
                 <state_interface name="velocity"/>
-            </joint> -->
+            </joint>
         </ros2_control>
     </xacro:macro>
